File: io.kicad_sch (KiCad schematic)
At the start: 15 parts, among them J14 D IN1, J15 D IN2, J16 D IN3

Commit message: Add title to all schematics pages
Other:
- title: (none) -> IO
Changed lines of the file:
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@@
 	(paper "A4")
 	(title_block
+		(title "IO")
 		(rev "1")
 	)

Commit message: Add power out to the digital inputs
Closes #18
Parts:
- J14, J15, J16: footprint Connector_JST:JST_PH_S2B-PH-K_1x02_P2.00mm_Horizontal -> Connector_JST:JST_PH_S3B-PH-K_1x03_P2.00mm_Horizontal; symbol Connector_Generic:Conn_01x02 -> Connector_Generic:Conn_01x03; LCSC C173752 -> C157929
Connections:
- net +3.3V: now also J14.1 (Pin_1), J15.1 (Pin_1), J16.1 (Pin_1)
- net at L13.1: now also J16.3 (Pin_3); no longer J16.2 (Pin_2)
- net at L10.1: now also J15.2 (Pin_2); no longer J15.1 (Pin_1)
- net at L11.1: now also J15.3 (Pin_3); no longer J15.2 (Pin_2)
- net at L12.1: now also J16.2 (Pin_2); no longer J16.1 (Pin_1)
- net at L8.1: now also J14.2 (Pin_2); no longer J14.1 (Pin_1)
- net at L9.1: now also J14.3 (Pin_3); no longer J14.2 (Pin_2)
