File: io.kicad_sch (KiCad schematic)
At the start: 17 parts, among them J14 D IN1, J15 D IN2, J16 D IN3, J22 1-Wire

Commit message: Add Reverse polarity protection
Closes #55
Connections:
- net +5V is gone; now on net +3.3V: J22.1 (Pin_1), R78.2
Changed lines of the file:
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@@
-	)
-	(symbol
-		(lib_id "power:+5V")
-		(at 177.8 21.59 0)
-		(unit 1)
-		(exclude_from_sim no)
-		(in_bom yes)
-		(on_board yes)
-		(dnp no)
-		(fields_autoplaced yes)
-		(property "Reference" "#PWR090"
-			(at 177.8 25.4 0)
-			(effects
-				(font
-					(size 1.27 1.27)
-				)
-				(hide yes)
-			)
-		)
-		(property "Value" "+5V"
-			(at 177.8 16.51 0)
-			(effects
-				(font
-					(size 1.27 1.27)
-				)
-			)
-		)
-		(property "Footprint" ""
-			(at 177.8 21.59 0)
-			(effects
-				(font
-					(size 1.27 1.27)
-				)
-				(hide yes)
-			)
-		)
-		(property "Datasheet" ""
-			(at 177.8 21.59 0)
-			(effects
-				(font
-					(size 1.27 1.27)
-				)
-				(hide yes)
-			)
-		)
-		(property "Description" "Power symbol creates a global label with name \"+5V\""
-			(at 177.8 21.59 0)
-			(effects
-				(font
-					(size 1.27 1.27)
-				)
-				(hide yes)
-			)
-		)
-		(pin "1"
-		)
-		(instances
-			(project "HydroponicFlowerControl"
-				(path "/b3c8a28b-9ce1-4002-b8e8-ef8cb73fe031/db02ea94-c311-42b2-be33-1b082fcd52fb"
-					(reference "#PWR090")
-					(unit 1)
-				)
-			)
-		)
 	)
 	(symbol
@@
 					(unit 1)
 				)
+			)
+		)
+	)
+	(symbol
+		(lib_id "power:+3.3V")
+		(at 177.8 21.59 0)
+		(unit 1)
+		(exclude_from_sim no)
+		(in_bom yes)
+		(on_board yes)
+		(dnp no)
+		(property "Reference" "#PWR0160"
+			(at 177.8 25.4 0)
+			(effects
+				(font
+					(size 1.27 1.27)
+				)
+				(hide yes)
+			)
+		)
+		(property "Value" "+3.3V"
+			(at 172.974 21.082 0)
+			(effects
+				(font
+					(size 1.27 1.27)
+				)
+			)
+		)
+		(property "Footprint" ""
+			(at 177.8 21.59 0)
+			(effects
+				(font
+					(size 1.27 1.27)
+				)
+				(hide yes)
+			)
+		)
+		(property "Datasheet" ""
+			(at 177.8 21.59 0)
+			(effects
+				(font
+					(size 1.27 1.27)
+				)
+				(hide yes)
+			)
+		)
+		(property "Description" "Power symbol creates a global label with name \"+3.3V\""
+			(at 177.8 21.59 0)
+			(effects
+				(font
+					(size 1.27 1.27)
+				)
+				(hide yes)
+			)
+		)
+		(pin "1"
+		)
+		(instances
+			(project "HydroponicFlowerControl"
+				(path "/b3c8a28b-9ce1-4002-b8e8-ef8cb73fe031/db02ea94-c311-42b2-be33-1b082fcd52fb"
+					(reference "#PWR0160")
+					(unit 1)
+				)

Commit message: Update fabrication properties
Parts:
- J14: value D IN1 -> S3B-PH-K-S(LF)(SN)
- J15: value D IN2 -> S3B-PH-K-S(LF)(SN)
- J16: value D IN3 -> S3B-PH-K-S(LF)(SN)
- J22: now not fitted; now in the parts list
Changed lines of the file:
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@@
 			)
 		)
-		(property "Value" "D IN2"
+		(property "Value" "S3B-PH-K-S(LF)(SN)"
 			(at 264.16 68.5799 0)
 			(hide yes)
@@
 			)
 		)
-		(property "Description" "Generic connector, single row, 01x03, script generated (kicad-library-utils/schlib/autogen/connector/)"
+		(property "Description" "D IN2"
 			(at 261.62 66.04 0)
 			(hide yes)
@@
 			)
 		)
-		(property "Value" "D IN1"
+		(property "Value" "S3B-PH-K-S(LF)(SN)"
 			(at 264.16 39.3699 0)
 			(hide yes)
@@
 			)
 		)
-		(property "Description" "Generic connector, single row, 01x03, script generated (kicad-library-utils/schlib/autogen/connector/)"
+		(property "Description" "D IN1"
 			(at 261.62 36.83 0)
 			(hide yes)
@@
 			)
 		)
-		(property "Value" "D IN3"
+		(property "Value" "S3B-PH-K-S(LF)(SN)"
 			(at 264.16 99.0599 0)
 			(hide yes)
@@
 			)
 		)
-		(property "Description" "Generic connector, single row, 01x03, script generated (kicad-library-utils/schlib/autogen/connector/)"
+		(property "Description" "D IN3"
 			(at 261.62 96.52 0)
 			(hide yes)
@@
 		(body_style 1)
 		(exclude_from_sim no)
-		(in_bom no)
-		(on_board yes)
-		(in_pos_files yes)
-		(dnp no)
+		(in_bom yes)
+		(on_board yes)
+		(in_pos_files yes)
+		(dnp yes)
 		(fields_autoplaced yes)
 		(property "Reference" "J22"

Commit message: Update fabrication properties
Parts:
- J14, J15, J16: FT Rotation Offset (none) -> 180; JLCPCB Position Offset 0,2 -> (none); JLCPCB Rotation Offset 180 -> (none)
Changed lines of the file:
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@@
 			)
 		)
-		(property "JLCPCB Rotation Offset" "180"
-			(at 261.62 66.04 0)
-			(hide yes)
-			(show_name no)
-			(do_not_autoplace no)
-			(effects
-				(font
-					(size 1.27 1.27)
-				)
-			)
-		)
-		(property "JLCPCB Position Offset" "0,2"
+		(property "FT Rotation Offset" "180"
 			(at 261.62 66.04 0)
 			(hide yes)
@@
 			)
 		)
-		(property "JLCPCB Rotation Offset" "180"
-			(at 261.62 36.83 0)
-			(hide yes)
-			(show_name no)
-			(do_not_autoplace no)
-			(effects
-				(font
-					(size 1.27 1.27)
-				)
-			)
-		)
-		(property "JLCPCB Position Offset" "0,2"
+		(property "FT Rotation Offset" "180"
 			(at 261.62 36.83 0)
 			(hide yes)
@@
 			)
 		)
-		(property "JLCPCB Rotation Offset" "180"
+		(property "FT Rotation Offset" "180"
 			(at 261.62 96.52 0)
 			(hide yes)
-			(show_name no)
-			(do_not_autoplace no)
-			(effects
-				(font
-					(size 1.27 1.27)
-				)
-			)
-		)
-		(property "JLCPCB Position Offset" "0,2"
-			(at 261.62 96.52 0)
-			(hide yes)
