File: flow_control.kicad_sch (KiCad schematic)
At the start: 56 parts, among them J10 Pump 1, J11 Temperature, J12 Pump 2, J13 Pump 3, J3 Flow, J7 Valve 1, J8 Valve 2, J9 Valve 3, U10 TPS4H160BQPWPRQ1, U11 TPS4H160BQPWPRQ1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

Commit message: Update fabrication properties
Parts:
- J10: value Pump 1 -> PhoenixContact_MC_1,5_2-G-3.81
- J11: value Temperature -> S2B-XH-A(LF)(SN)
- J12: value Pump 2 -> PhoenixContact_MC_1,5_2-G-3.81
- J13: value Pump 3 -> PhoenixContact_MC_1,5_2-G-3.81
- J3: value Flow -> S3B-XH-A(LF)(SN)
- J7: value Valve 1 -> S2B-XH-A(LF)(SN)
- J8: value Valve 2 -> S2B-XH-A(LF)(SN)
- J9: value Valve 3 -> S3B-XH-A(LF)(SN)
Changed lines of the file:
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@@
 			)
 		)
-		(property "Value" "Pump 2"
+		(property "Value" "PhoenixContact_MC_1,5_2-G-3.81"
 			(at 179.07 148.5899 0)
 			(hide yes)
@@
 			)
 		)
-		(property "Description" "Generic screw terminal, single row, 01x02, script generated (kicad-library-utils/schlib/autogen/connector/)"
+		(property "Description" "Pump 2"
 			(at 176.53 146.05 0)
 			(hide yes)
@@
 			)
 		)
-		(property "Value" "Pump 3"
+		(property "Value" "PhoenixContact_MC_1,5_2-G-3.81"
 			(at 203.2 139.6999 0)
 			(hide yes)
@@
 			)
 		)
-		(property "Description" "Generic screw terminal, single row, 01x02, script generated (kicad-library-utils/schlib/autogen/connector/)"
+		(property "Description" "Pump 3"
 			(at 200.66 137.16 0)
 			(hide yes)
@@
 			)
 		)
-		(property "Value" "Valve 2"
+		(property "Value" "S2B-XH-A(LF)(SN)"
 			(at 147.32 58.4199 0)
 			(hide yes)
@@
 			)
 		)
-		(property "Description" "Generic connector, single row, 01x02, script generated (kicad-library-utils/schlib/autogen/connector/)"
+		(property "Description" "Valve 2"
 			(at 144.78 55.88 0)
 			(hide yes)
@@
 			)
 		)
-		(property "Value" "Valve 1"
+		(property "Value" "S2B-XH-A(LF)(SN)"
 			(at 147.32 49.5299 0)
 			(hide yes)
@@
 			)
 		)
-		(property "Description" "Generic connector, single row, 01x02, script generated (kicad-library-utils/schlib/autogen/connector/)"
+		(property "Description" "Valve 1"
 			(at 144.78 46.99 0)
 			(hide yes)
@@
 			)
 		)
-		(property "Value" "Temperature"
+		(property "Value" "S2B-XH-A(LF)(SN)"
 			(at 270.51 82.5499 0)
 			(hide yes)
@@
 			)
 		)
-		(property "Description" "Generic connector, single row, 01x02, script generated (kicad-library-utils/schlib/autogen/connector/)"
+		(property "Description" "Temperature"
 			(at 267.97 80.01 0)
 			(hide yes)
@@
 			)
 		)
-		(property "Value" "Flow"
+		(property "Value" "S3B-XH-A(LF)(SN)"
 			(at 270.51 36.8299 0)
 			(hide yes)
@@
 			)
 		)
-		(property "Description" "Generic connector, single row, 01x03, script generated (kicad-library-utils/schlib/autogen/connector/)"
+		(property "Description" "Flow"
 			(at 267.97 35.56 0)
 			(hide yes)
@@
 			)
 		)
-		(property "Value" "Pump 1"
+		(property "Value" "PhoenixContact_MC_1,5_2-G-3.81"
 			(at 153.67 157.4799 0)
 			(hide yes)
@@
 			)
 		)
-		(property "Description" "Generic screw terminal, single row, 01x02, script generated (kicad-library-utils/schlib/autogen/connector/)"
+		(property "Description" "Pump 1"
 			(at 151.13 154.94 0)
 			(hide yes)
@@
 			)
 		)
-		(property "Value" "Valve 3"
+		(property "Value" "S3B-XH-A(LF)(SN)"
 			(at 152.4 86.3599 0)
 			(hide yes)
@@
 			)
 		)
-		(property "Description" "Generic connector, single row, 01x03, script generated (kicad-library-utils/schlib/autogen/connector/)"
+		(property "Description" "Valve 3"
 			(at 149.86 85.09 0)
 			(hide yes)

Commit message: Update fabrication properties
Parts:
- J10, J12, J13: JLCPCB Position Offset 0,3 -> (none)
- J11, J3, J7, J8, J9: FT Rotation Offset (none) -> 180; JLCPCB Position Offset 0,3.5 -> (none); JLCPCB Rotation Offset 180 -> (none)
Changed lines of the file:
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@@
 			)
 		)
-		(property "LCSC alt" ""
-			(at 176.53 146.05 0)
-			(hide yes)
-			(show_name no)
-			(do_not_autoplace no)
-			(effects
-				(font
-					(size 1.27 1.27)
-				)
-			)
-		)
-		(property "JLCPCB Position Offset" "0,3"
-			(at 176.53 146.05 0)
-			(hide yes)
-			(show_name no)
-			(do_not_autoplace no)
-			(effects
-				(font
-					(size 1.27 1.27)
-				)
-			)
-		)
 		(pin "2"
 		)
@@
 			)
 		)
-		(property "LCSC alt" ""
-			(at 200.66 137.16 0)
-			(hide yes)
-			(show_name no)
-			(do_not_autoplace no)
-			(effects
-				(font
-					(size 1.27 1.27)
-				)
-			)
-		)
-		(property "JLCPCB Position Offset" "0,3"
-			(at 200.66 137.16 0)
-			(hide yes)
-			(show_name no)
-			(do_not_autoplace no)
-			(effects
-				(font
-					(size 1.27 1.27)
-				)
-			)
-		)
 		(pin "2"
 		)
@@
 			)
 		)
-		(property "LCSC alt" ""
-			(at 144.78 55.88 0)
-			(hide yes)
-			(show_name no)
-			(do_not_autoplace no)
-			(effects
-				(font
-					(size 1.27 1.27)
-				)
-			)
-		)
-		(property "JLCPCB Position Offset" "0,3.5"
-			(at 144.78 55.88 0)
-			(hide yes)
-			(show_name no)
-			(do_not_autoplace no)
-			(effects
-				(font
-					(size 1.27 1.27)
-				)
-			)
-		)
-		(property "JLCPCB Rotation Offset" "180"
+		(property "FT Rotation Offset" "180"
 			(at 144.78 55.88 0)
 			(hide yes)
@@
 			)
 		)
-		(property "LCSC alt" ""
-			(at 144.78 46.99 0)
-			(hide yes)
-			(show_name no)
-			(do_not_autoplace no)
-			(effects
-				(font
-					(size 1.27 1.27)
-				)
-			)
-		)
-		(property "JLCPCB Position Offset" "0,3.5"
-			(at 144.78 46.99 0)
-			(hide yes)
-			(show_name no)
-			(do_not_autoplace no)
-			(effects
-				(font
-					(size 1.27 1.27)
-				)
-			)
-		)
-		(property "JLCPCB Rotation Offset" "180"
+		(property "FT Rotation Offset" "180"
 			(at 144.78 46.99 0)
 			(hide yes)
@@
 			)
 		)
-		(property "JLCPCB Position Offset" "0,3.5"
-			(at 267.97 80.01 0)
-			(hide yes)
-			(show_name no)
-			(do_not_autoplace no)
-			(effects
-				(font
-					(size 1.27 1.27)
-				)
-			)
-		)
-		(property "JLCPCB Rotation Offset" "180"
+		(property "FT Rotation Offset" "180"
 			(at 267.97 80.01 0)
 			(hide yes)
@@
 			)
 		)
-		(property "JLCPCB Position Offset" "0,3.5"
-			(at 267.97 35.56 0)
-			(hide yes)
-			(show_name no)
-			(do_not_autoplace no)
-			(effects
-				(font
-					(size 1.27 1.27)
-				)
-			)
-		)
-		(property "JLCPCB Rotation Offset" "180"
+		(property "FT Rotation Offset" "180"
 			(at 267.97 35.56 0)
 			(hide yes)
@@
 			)
 		)
-		(property "LCSC alt" ""
-			(at 151.13 154.94 0)
-			(hide yes)
-			(show_name no)
-			(do_not_autoplace no)
-			(effects
-				(font
-					(size 1.27 1.27)
-				)
-			)
-		)
-		(property "JLCPCB Position Offset" "0,3"
-			(at 151.13 154.94 0)
-			(hide yes)
-			(show_name no)
-			(do_not_autoplace no)
-			(effects
-				(font
-					(size 1.27 1.27)
-				)
-			)
-		)
 		(pin "2"
 		)
@@
 			)
 		)
-		(property "LCSC alt" ""
-			(at 149.86 85.09 0)
-			(hide yes)
-			(show_name no)
-			(do_not_autoplace no)
-			(effects
-				(font
-					(size 1.27 1.27)
-				)
-			)
-		)
 		(property "LCSC" "C157928"
 			(at 149.86 85.09 0)
@@
 			)
 		)
-		(property "JLCPCB Position Offset" "0,3.5"
-			(at 149.86 85.09 0)
-			(hide yes)
-			(show_name no)
-			(do_not_autoplace no)
-			(effects
-				(font
-					(size 1.27 1.27)
-				)
-			)
-		)
-		(property "JLCPCB Rotation Offset" "180"
+		(property "FT Rotation Offset" "180"
 			(at 149.86 85.09 0)
 			(hide yes)
