File: rpi.kicad_sch (KiCad schematic)
At the start: 15 parts, among them J18 Raspberry_Pi_2_3, U1 AT24C256C, U16 MCP2518FD-xQBB, U19 SN65HVD230, Y2 40MHz

Commit message: Update fabrication properties
Parts:
- J18, U19: FT Rotation Offset (none) -> 0; JLCPCB Rotation Offset 0 -> (none)
Changed lines of the file:
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@@
 			)
 		)
-		(property "JLCPCB Rotation Offset" "0"
-			(at 257.81 134.62 0)
-			(hide yes)
-			(show_name no)
-			(do_not_autoplace no)
-			(effects
-				(font
-					(size 1.27 1.27)
-				)
-			)
-		)
-		(property "LCSC alt" ""
+		(property "FT Rotation Offset" "0"
 			(at 257.81 134.62 0)
 			(hide yes)
@@
 			)
 		)
-		(property "JLCPCB Rotation Offset" "0"
+		(property "FT Rotation Offset" "0"
 			(at 66.04 63.5 0)
 			(hide yes)
@@
 			(at 209.55 137.16 0)
 			(hide yes)
-			(show_name no)
-			(do_not_autoplace no)
-			(effects
-				(font
-					(size 1.27 1.27)
-				)
-			)
-		)
-		(property "LCSC alt" ""
-			(at 209.55 137.16 0)
-			(hide yes)
